Commit message: final_data

File: agentsd_ws/install/smart_agent_gazebo/share/smart_agent_gazebo/urdf/smart_agent.urdf.xacro (robot description, xacro)
@@ -1 +1,203 @@
-/home/test/wf3/gazebo/agentsd_ws/build/smart_agent_gazebo/urdf/smart_agent.urdf.xacro
+<?xml version="1.0"?>
+<robot name="smart_agent" xmlns:xacro="http://www.ros.org/wiki/xacro">
+  <link name="base_link">
+    <inertial>
+      <origin xyz="0 0 0" rpy="0 0 0"/>
+      <mass value="8.0"/>
+      <inertia ixx="0.28" ixy="0.0" ixz="0.0" iyy="0.28" iyz="0.0" izz="0.45"/>
+    </inertial>
+    <visual>
+      <origin xyz="0 0 0.24" rpy="0 0 0"/>
+      <geometry>
+        <box size="0.5 0.35 0.48"/>
+      </geometry>
+      <material name="gray">
+        <color rgba="0.5 0.5 0.5 1"/>
+      </material>
+    </visual>
+    <collision>
+      <origin xyz="0 0 0.24" rpy="0 0 0"/>
+      <geometry>
+        <box size="0.5 0.35 0.48"/>
+      </geometry>
+    </collision>
+  </link>
+  <link name="lidar_link">
+    <visual>
+      <geometry>
+        <cylinder length="0.04" radius="0.04"/>
+      </geometry>
+      <material name="black">
+        <color rgba="0.1 0.1 0.1 1"/>
+      </material>
+    </visual>
+  </link>
+  <joint name="lidar_joint" type="fixed">
+    <parent link="base_link"/>
+    <child link="lidar_link"/>
+    <origin xyz="0.10 0 0.56" rpy="0 0 0"/>
+  </joint>
+  <link name="front_camera_link">
+    <visual>
+      <geometry>
+        <box size="0.05 0.05 0.05"/>
+      </geometry>
+      <material name="blue">
+        <color rgba="0.2 0.2 0.9 1"/>
+      </material>
+    </visual>
+  </link>
+  <joint name="front_camera_joint" type="fixed">
+    <parent link="base_link"/>
+    <child link="front_camera_link"/>
+    <origin xyz="0.23 0 0.50" rpy="0 0 0"/>
+  </joint>
+  <link name="rear_camera_link">
+    <visual>
+      <geometry>
+        <box size="0.05 0.05 0.05"/>
+      </geometry>
+      <material name="green">
+        <color rgba="0.2 0.8 0.2 1"/>
+      </material>
+    </visual>
+  </link>
+  <joint name="rear_camera_joint" type="fixed">
+    <parent link="base_link"/>
+    <child link="rear_camera_link"/>
+    <origin xyz="-0.23 0 0.50" rpy="0 0 3.14159"/>
+  </joint>
+  <link name="depth_camera_link">
+    <visual>
+      <geometry>
+        <box size="0.05 0.05 0.05"/>
+      </geometry>
+      <material name="orange">
+        <color rgba="0.9 0.4 0.1 1"/>
+      </material>
+    </visual>
+  </link>
+  <joint name="depth_camera_joint" type="fixed">
+    <parent link="base_link"/>
+    <child link="depth_camera_link"/>
+    <origin xyz="0.23 0 0.50" rpy="0 0 0"/>
+  </joint>
+  <gazebo reference="base_link">
+    <material>Gazebo/Grey</material>
+  </gazebo>
+  <gazebo reference="lidar_link">
+    <sensor type="ray" name="lidar_sensor">
+      <always_on>true</always_on>
+      <update_rate>10</update_rate>
+      <visualize>true</visualize>
+      <pose>0 0 0 0 0 0</pose>
+      <ray>
+        <scan>
+          <horizontal>
+            <samples>720</samples>
+            <resolution>1</resolution>
+            <min_angle>-3.14159</min_angle>
+            <max_angle>3.14159</max_angle>
+          </horizontal>
+        </scan>
+        <range>
+          <min>0.12</min>
+          <max>15.0</max>
+          <resolution>0.01</resolution>
+        </range>
+        <noise>
+          <type>gaussian</type>
+          <mean>0.0</mean>
+          <stddev>0.005</stddev>
+        </noise>
+      </ray>
+      <plugin name="gazebo_ros_lidar" filename="libgazebo_ros_ray_sensor.so">
+        <ros>
+          <namespace>/agent</namespace>
+          <remapping>~/out:=/agent/lidar/scan</remapping>
+        </ros>
+        <frame_name>lidar_link</frame_name>
+      </plugin>
+    </sensor>
+  </gazebo>
+  <gazebo reference="front_camera_link">
+    <sensor type="camera" name="front_rgb_sensor">
+      <always_on>true</always_on>
+      <update_rate>20</update_rate>
+      <camera>
+        <horizontal_fov>1.396</horizontal_fov>
+        <image>
+          <width>640</width>
+          <height>480</height>
+          <format>R8G8B8</format>
+        </image>
+        <clip>
+          <near>0.05</near>
+          <far>50.0</far>
+        </clip>
+      </camera>
+      <plugin name="gazebo_ros_front_camera" filename="libgazebo_ros_camera.so">
+        <ros>
+          <namespace>/agent</namespace>
+          <remapping>image_raw:=/agent/front_camera/image_raw</remapping>
+          <remapping>camera_info:=/agent/front_camera/camera_info</remapping>
+        </ros>
+        <frame_name>front_camera_link</frame_name>
+      </plugin>
+    </sensor>
+  </gazebo>
+  <gazebo reference="rear_camera_link">
+    <sensor type="camera" name="rear_rgb_sensor">
+      <always_on>true</always_on>
+      <update_rate>20</update_rate>
+      <camera>
+        <horizontal_fov>1.396</horizontal_fov>
+        <image>
+          <width>640</width>
+          <height>480</height>
+          <format>R8G8B8</format>
+        </image>
+        <clip>
+          <near>0.05</near>
+          <far>50.0</far>
+        </clip>
+      </camera>
+      <plugin name="gazebo_ros_rear_camera" filename="libgazebo_ros_camera.so">
+        <ros>
+          <namespace>/agent</namespace>
+          <remapping>image_raw:=/agent/rear_camera/image_raw</remapping>
+          <remapping>camera_info:=/agent/rear_camera/camera_info</remapping>
+        </ros>
+        <frame_name>rear_camera_link</frame_name>
+      </plugin>
+    </sensor>
+  </gazebo>
+  <gazebo reference="depth_camera_link">
+    <sensor type="depth" name="depth_sensor">
+      <always_on>true</always_on>
+      <update_rate>15</update_rate>
+      <camera>
+        <horizontal_fov>1.396</horizontal_fov>
+        <image>
+          <width>640</width>
+          <height>480</height>
+          <format>R8G8B8</format>
+        </image>
+        <clip>
+          <near>0.1</near>
+          <far>20.0</far>
+        </clip>
+      </camera>
+      <plugin name="gazebo_ros_depth_camera" filename="libgazebo_ros_camera.so">
+        <ros>
+          <namespace>/agent</namespace>
+          <remapping>image_raw:=/agent/depth_camera/image_raw</remapping>
+          <remapping>camera_info:=/agent/depth_camera/camera_info</remapping>
+          <remapping>depth/image_raw:=/agent/depth_camera/depth/image_raw</remapping>
+          <remapping>points:=/agent/depth_camera/points</remapping>
+        </ros>
+        <frame_name>depth_camera_link</frame_name>
+      </plugin>
+    </sensor>
+  </gazebo>
+</robot>
